Commit message: added optical camera link to my_robot.xarco

File: my_robot/urdf/my_robot.xacro (robot description, xacro)
@@ -176,4 +176,11 @@
     <axis xyz="0 1 0" rpy="0 0 0"/>
   </joint>
+  <joint type="fixed" name="camera_optical_joint">
+    <origin xyz="0 0 0" rpy="-1.5707 0 -1.5707" />
+    <parent link="camera_link" />
+    <child link="camera_link_optical" />
+  </joint>
+  <link name="camera_link_optical">
+  </link>
   <gazebo reference='chassis'>
     <material>Gazebo/Blue</material>

Commit message: Fixed broken child link in my_robot.xacro

File: my_robot/urdf/my_robot.xacro (robot description, xacro)
@@ -178,5 +178,5 @@
   <joint type="fixed" name="camera_optical_joint">
     <origin xyz="0 0 0" rpy="-1.5707 0 -1.5707" />
-    <parent link="camera_link" />
+    <parent link="camera" />
     <child link="camera_link_optical" />
   </joint>
